File: eagle_board/odd_v1.1/odd_v1.sch (EAGLE design)
At the start: 17 parts

Commit message: Modified board, there were accidental and dumb connections being made. Also added two capacitors for use with the voltage regulator.
Parts:
- added C1, C2: (no value), resistor:C-US075-032X103
- U$1, U$2, U$3, U$4, U$5: value CREESMDRGBLED6PADSMD -> RGBLED
Connections:
- net N$18: now also C1.1
- net N$19: now also C1.2, C2.1
- net N$22: now also C2.2
Changed lines of the file:
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@@
 <?xml version="1.0" encoding="utf-8"?>
 <!DOCTYPE eagle SYSTEM "eagle.dtd">
-<eagle version="6.4">
+<eagle version="6.3">
 <drawing>
 <settings>
@@
 <parts>
 <part name="IC1" library="tcl5940" deviceset="TCL5940" device=""/>
-<part name="U$1" library="odd_led" deviceset="CREESMDRGBLED" device="6PADSMD"/>
-<part name="U$2" library="odd_led" deviceset="CREESMDRGBLED" device="6PADSMD"/>
-<part name="U$3" library="odd_led" deviceset="CREESMDRGBLED" device="6PADSMD"/>
-<part name="U$4" library="odd_led" deviceset="CREESMDRGBLED" device="6PADSMD"/>
-<part name="U$5" library="odd_led" deviceset="CREESMDRGBLED" device="6PADSMD"/>
+<part name="U$1" library="odd_led" deviceset="CREESMDRGBLED" device="6PADSMD" value="RGBLED"/>
+<part name="U$2" library="odd_led" deviceset="CREESMDRGBLED" device="6PADSMD" value="RGBLED"/>
+<part name="U$3" library="odd_led" deviceset="CREESMDRGBLED" device="6PADSMD" value="RGBLED"/>
+<part name="U$4" library="odd_led" deviceset="CREESMDRGBLED" device="6PADSMD" value="RGBLED"/>
+<part name="U$5" library="odd_led" deviceset="CREESMDRGBLED" device="6PADSMD" value="RGBLED"/>
 <part name="U$17" library="ODD_LDO" deviceset="ODD_LDO" device="ODDLDO"/>
 <part name="R1" library="resistor" deviceset="R-US_" device="0204/7"/>
@@
 <part name="GND" library="wirepad" deviceset="2,54/1,1" device=""/>
 <part name="SOUT" library="wirepad" deviceset="2,54/1,1" device=""/>
+<part name="C1" library="resistor" deviceset="C-US" device="075-032X103"/>
+<part name="C2" library="resistor" deviceset="C-US" device="075-032X103"/>
 </parts>
 <sheets>
@@
 <instance part="GND" gate="1" x="111.76" y="25.4" rot="R180"/>
 <instance part="SOUT" gate="1" x="81.28" y="-30.48" rot="R90"/>
+<instance part="C1" gate="G$1" x="99.06" y="45.72"/>
+<instance part="C2" gate="G$1" x="88.9" y="40.64"/>
 </instances>
 <busses>
@@
 <pinref part="U$17" gate="G$1" pin="INPUT"/>
 <wire x1="109.22" y1="55.88" x2="101.6" y2="55.88" width="0.1524" layer="91"/>
-<wire x1="101.6" y1="55.88" x2="101.6" y2="43.18" width="0.1524" layer="91"/>
+<wire x1="101.6" y1="55.88" x2="101.6" y2="48.26" width="0.1524" layer="91"/>
+<pinref part="C1" gate="G$1" pin="1"/>
+<wire x1="101.6" y1="48.26" x2="101.6" y2="43.18" width="0.1524" layer="91"/>
+<wire x1="99.06" y1="48.26" x2="101.6" y2="48.26" width="0.1524" layer="91"/>
+<junction x="101.6" y="48.26"/>
 </segment>
 </net>
@@
 <wire x1="71.12" y1="45.72" x2="83.82" y2="45.72" width="0.1524" layer="91"/>
 <wire x1="83.82" y1="45.72" x2="91.44" y2="45.72" width="0.1524" layer="91"/>
-<wire x1="91.44" y1="45.72" x2="91.44" y2="38.1" width="0.1524" layer="91"/>
-<wire x1="91.44" y1="38.1" x2="101.6" y2="38.1" width="0.1524" layer="91"/>
+<wire x1="91.44" y1="45.72" x2="91.44" y2="43.18" width="0.1524" layer="91"/>
+<wire x1="91.44" y1="43.18" x2="91.44" y2="38.1" width="0.1524" layer="91"/>
+<wire x1="91.44" y1="38.1" x2="99.06" y2="38.1" width="0.1524" layer="91"/>
 <junction x="101.6" y="38.1"/>
 <pinref part="R1" gate="G$1" pin="2"/>
+<wire x1="99.06" y1="38.1" x2="101.6" y2="38.1" width="0.1524" layer="91"/>
 <wire x1="78.74" y1="30.48" x2="83.82" y2="30.48" width="0.1524" layer="91"/>
 <wire x1="83.82" y1="30.48" x2="83.82" y2="45.72" width="0.1524" layer="91"/>
@@
 <wire x1="71.12" y1="58.42" x2="71.12" y2="45.72" width="0.1524" layer="91"/>
 <junction x="71.12" y="45.72"/>
+<pinref part="C1" gate="G$1" pin="2"/>
+<wire x1="99.06" y1="40.64" x2="99.06" y2="38.1" width="0.1524" layer="91"/>
+<junction x="99.06" y="38.1"/>
+<pinref part="C2" gate="G$1" pin="1"/>
+<wire x1="88.9" y1="43.18" x2="91.44" y2="43.18" width="0.1524" layer="91"/>
+<junction x="91.44" y="43.18"/>
 </segment>
 </net>
@@
 <wire x1="-45.72" y1="-15.24" x2="-45.72" y2="2.54" width="0.1524" layer="91"/>
 <junction x="-45.72" y="2.54"/>
-</segment>
-</net>
+<pinref part="C2" gate="G$1" pin="2"/>
+<wire x1="88.9" y1="35.56" x2="88.9" y2="33.02" width="0.1524" layer="91"/>
+</segment>
+</net>
